Commit message: Update model parameters. Cleaned code and moved dependencies

File: tacbot_description/urdf/kinect.xacro (robot description, xacro)
@@ -2,13 +2,13 @@
 <robot name="sensor_kinect" xmlns:xacro="http://ros.org/wiki/xacro">
   <xacro:property name="kinect_cam_py" value="-0.0125"/>
-	<xacro:property name="cam_px" value="-0.087" />
-<!--	<property name="cam_py" value="-0.0125" /> -->
-	<xacro:property name="cam_pz" value="0.12" />
+        <xacro:property name="cam_px" value="0.085" />
+        <xacro:property name="cam_py" value="0.0125" />
+        <xacro:property name="cam_pz" value="0.14" />
 	<xacro:property name="cam_or" value="0" />
 	<xacro:property name="cam_op" value="0" />
-	<xacro:property name="cam_oy" value="0" />
+        <xacro:property name="cam_oy" value="${pi}" />
   <xacro:macro name="sensor_kinect" params="parent">
     <joint name="camera_rgb_joint" type="fixed">
-      <origin xyz="${cam_px} ${kinect_cam_py} ${cam_pz}" rpy="${cam_or} ${cam_op} ${cam_oy}"/>
+      <origin xyz="${cam_px} ${cam_py} ${cam_pz}" rpy="${cam_or} ${cam_op} ${cam_oy}"/>
       <parent link="${parent}"/>
       <child link="camera_rgb_frame" />

File: tacbot_description/urdf/robot.xacro (robot description, xacro)
@@ -1,12 +1,12 @@
 <?xml version="1.0"?>
 <!-- Tacbot robot -->
-<robot name="tacbot" xmlns:xacro="http://www.ros.org/wiki/xacro">
+<robot name="tacbot" xmlns:xacro="http://ros.org/wiki/xacro">
     <!-- Constants-->
-    <xacro:property name="base_length"  value=".35"/>
-    <xacro:property name="base_width"   value=".3"/>
-    <xacro:property name="base_height"  value=".055"/>
-    <xacro:property name="wheel_width"  value=".04"/>
-    <xacro:property name="wheel_radius" value=".06"/>
-    <xacro:property name="wheel_dis"    value=".02"/>
+    <xacro:property name="base_length"  value=".297"/>
+    <xacro:property name="base_width"   value=".189"/>
+    <xacro:property name="base_height"  value=".06"/>
+    <xacro:property name="wheel_width"  value=".055"/>
+    <xacro:property name="wheel_radius" value=".055"/>
+    <xacro:property name="wheel_dis"    value=".0235"/>
     <!-- Base dummy link -->
     <link name="base_footprint"/>
@@ -26,5 +26,5 @@
             <xacro:base_origin/>
             <material name="gray">
-                         <color rgba=".2 .2 .2 1" />
+                <color rgba=".2 .2 .2 1" />
             </material>
         </visual>
@@ -34,24 +34,17 @@
             </geometry>
             <xacro:base_origin/>
-            <contact_coefficients mu="0" kp="1000.0" kd="1.0"/>
         </collision>
         <inertial>
-                      <origin xyz="0 0 0"/>
-            <mass value="3"/> <!-- 3 kg -->
-            <inertia ixx="0.3" ixy="0" ixz="0" iyy="0.3" iyz="0" izz="0.6" />
+            <mass value="4"/> <!-- 4 kg -->
+            <origin xyz="0 0 0"/>
+            <inertia ixx="0.02" ixy="0" ixz="0" iyy="0.02" iyz="0" izz="0.03" />
         </inertial>
     </link>
-    <!-- Wheel macros -->
-    <xacro:macro name="wheel_cyl"> <cylinder radius="${wheel_radius}" length="${wheel_width}" /> </xacro:macro>
-    <xacro:macro name="wheel_joint_origin">
-        <origin xyz="${front*(base_length/2-wheel_dis)} ${side*(base_width/2+wheel_width/2)} ${wheel_radius}"
-                rpy="${pi/2} 0 0"/>
-    </xacro:macro>
+    <!-- Wheel links -->
     <xacro:macro name="wheel" params="postfix side front">
-        <!-- Wheel links -->
         <link name="wheel_${postfix}">
             <visual>
                 <geometry>
-                    <xacro:wheel_cyl />
+                    <cylinder radius="${wheel_radius}" length="${wheel_width}"/>
                 </geometry>
                 <origin xyz="0 0 0" rpy="0 0 0"/>
@@ -62,12 +55,11 @@
             <collision>
                 <geometry>
-                    <xacro:wheel_cyl />
+                    <cylinder radius="${wheel_radius}" length="${wheel_width}"/>
                 </geometry>
                 <origin xyz="0 0 0" rpy="0 0 0"/>
-                <contact_coefficients mu="0" kp="1000.0" kd="1.0"/>
             </collision>
             <inertial>
-                <mass value="0.1" />
-                <inertia ixx="0.05" ixy="0.0" ixz="0.0" iyy="0.05" iyz="0.0" izz="0.05"/>
+                <mass value="0.2" />
+                <inertia ixx="0.005" ixy="0.0" ixz="0.0" iyy="0.005" iyz="0.0" izz="0.005"/>
             </inertial>
         </link>
@@ -76,9 +68,10 @@
             <parent link="base_link"/>
             <child link="wheel_${postfix}"/>
-            <xacro:wheel_joint_origin />
+            <origin xyz="${front*(base_length/2-wheel_dis)} ${side*(base_width/2+wheel_width/2)} ${wheel_radius}"
+                    rpy="${pi/2} 0 0"/>
             <axis xyz="0 0 1"/>
             <dynamics damping="0" friction = "0" />
-            <limit effort="50" velocity="1.0" />
-            <safety_controller k_velocity="10" />
+            <limit effort="5" velocity="1.0" />
+            <safety_controller k_velocity="5" />
         </joint>
         <!-- Wheel transmissions -->

File: tacbot_description/urdf/robot_gazebo.xacro (robot description, xacro)
@@ -6,5 +6,5 @@
             <mu1>1.0</mu1>
             <mu2>1.0</mu2>
-            <kp>10000.0</kp>
+            <kp>100000.0</kp>
             <kd>10.0</kd>
             <minDepth>0.001</minDepth>
@@ -33,5 +33,5 @@
                 <wheel_FL_joint_name>wheel_FL_joint</wheel_FL_joint_name>
                 <wheel_FR_joint_name>wheel_FR_joint</wheel_FR_joint_name>
-                <reg_kp>1.0</reg_kp>
+                <reg_kp>2.0</reg_kp>
                 <reg_ki>0</reg_ki>
                 <reg_kd>0</reg_kd>
@@ -39,5 +39,5 @@
                 <front_wheel_separation>.3</front_wheel_separation>
                 <wheel_diameter>0.11</wheel_diameter>
-                <max_torque>0.5</max_torque>
+                <max_torque>0.4</max_torque>
                 <publish_tf>1</publish_tf>
             </plugin>

Commit message: Add robot_prefix parameter to launchers

File: tacbot_description/urdf/kinect.xacro (robot description, xacro)
@@ -8,23 +8,23 @@
 	<xacro:property name="cam_op" value="0" />
         <xacro:property name="cam_oy" value="${pi}" />
-  <xacro:macro name="sensor_kinect" params="parent">
-    <joint name="camera_rgb_joint" type="fixed">
+  <xacro:macro name="sensor_kinect" params="prefix parent">
+    <joint name="${prefix}_camera_rgb_joint" type="fixed">
       <origin xyz="${cam_px} ${cam_py} ${cam_pz}" rpy="${cam_or} ${cam_op} ${cam_oy}"/>
       <parent link="${parent}"/>
-      <child link="camera_rgb_frame" />
+      <child link="${prefix}_camera_rgb_frame" />
     </joint>
-    <link name="camera_rgb_frame"/>
-    <joint name="camera_rgb_optical_joint" type="fixed">
+    <link name="${prefix}_camera_rgb_frame"/>
+    <joint name="${prefix}_camera_rgb_optical_joint" type="fixed">
       <origin xyz="0 0 0" rpy="${-pi/2} 0 ${-pi/2}" />
-      <parent link="camera_rgb_frame" />
-      <child link="camera_rgb_optical_frame" />
+      <parent link="${prefix}_camera_rgb_frame" />
+      <child link="${prefix}_camera_rgb_optical_frame" />
     </joint>
-    <link name="camera_rgb_optical_frame"/>
-    <joint name="camera_joint" type="fixed">
+    <link name="${prefix}_camera_rgb_optical_frame"/>
+    <joint name="${prefix}_camera_joint" type="fixed">
       <origin xyz="-0.031 ${-kinect_cam_py} -0.016" rpy="0 0 0"/>
-      <parent link="camera_rgb_frame"/>
-      <child link="camera_link"/>
+      <parent link="${prefix}_camera_rgb_frame"/>
+      <child link="${prefix}_camera_link"/>
     </joint>
-      <link name="camera_link">
+      <link name="${prefix}_camera_link">
       <visual>
        <origin xyz="0 0 0" rpy="0 0 ${pi/2}"/>
@@ -48,16 +48,16 @@
     </link>
     <!-- For Gazebo simulation only -->
-	<joint name="camera_depth_joint" type="fixed">
+	<joint name="${prefix}_camera_depth_joint" type="fixed">
 	  <origin xyz="0 ${2 * -kinect_cam_py} 0" rpy="0 0 0" />
-	  <parent link="camera_rgb_frame" />
-	  <child link="camera_depth_frame" />
+	  <parent link="${prefix}_camera_rgb_frame" />
+	  <child link="${prefix}_camera_depth_frame" />
 	</joint>
-	<link name="camera_depth_frame"/>
-	<joint name="camera_depth_optical_joint" type="fixed">
+	<link name="${prefix}_camera_depth_frame"/>
+	<joint name="${prefix}_camera_depth_optical_joint" type="fixed">
 	  <origin xyz="0 0 0" rpy="${-pi/2} 0 ${-pi/2}" />
-	  <parent link="camera_depth_frame" />
-	  <child link="camera_depth_optical_frame" />
+	  <parent link="${prefix}_camera_depth_frame" />
+	  <child link="${prefix}_camera_depth_optical_frame" />
 	</joint>
-	<link name="camera_depth_optical_frame"/>
+	<link name="${prefix}_camera_depth_optical_frame"/>
   </xacro:macro>
 </robot>

File: tacbot_description/urdf/robot.xacro (robot description, xacro)
@@ -3,4 +3,5 @@
 <robot name="tacbot" xmlns:xacro="http://ros.org/wiki/xacro">
     <!-- Constants-->
+	 <xacro:property name="prefix"		 value="r1"/>
     <xacro:property name="base_length"  value=".297"/>
     <xacro:property name="base_width"   value=".189"/>
@@ -10,14 +11,14 @@
     <xacro:property name="wheel_dis"    value=".0235"/>
     <!-- Base dummy link -->
-    <link name="base_footprint"/>
-    <joint name="base_joint" type="fixed">
+    <link name="${prefix}_base_footprint"/>
+    <joint name="${prefix}_base_joint" type="fixed">
       <origin xyz="0 0 0.0" rpy="0 0 0" />
-      <parent link="base_footprint"/>
-      <child link="base_link" />
+      <parent link="${prefix}_base_footprint"/>
+      <child link="${prefix}_base_link" />
     </joint>
     <!-- Base link definition-->
     <xacro:macro name="base_box"> <box size="${base_length} ${base_width} ${base_height}"/> </xacro:macro>
     <xacro:macro name="base_origin"> <origin xyz="0 0 ${wheel_radius}" rpy="0 0 0"/> </xacro:macro>
-    <link name="base_link">
+    <link name="${prefix}_base_link">
         <visual>
             <geometry>
@@ -43,5 +44,5 @@
     <!-- Wheel links -->
     <xacro:macro name="wheel" params="postfix side front">
-        <link name="wheel_${postfix}">
+        <link name="${prefix}_wheel_${postfix}">
             <visual>
                 <geometry>
@@ -65,7 +66,7 @@
         </link>
         <!-- Wheel joints -->
-        <joint name="wheel_${postfix}_joint" type="continuous">
-            <parent link="base_link"/>
-            <child link="wheel_${postfix}"/>
+        <joint name="${prefix}_wheel_${postfix}_joint" type="continuous">
+            <parent link="${prefix}_base_link"/>
+            <child link="${prefix}_wheel_${postfix}"/>
             <origin xyz="${front*(base_length/2-wheel_dis)} ${side*(base_width/2+wheel_width/2)} ${wheel_radius}"
                     rpy="${pi/2} 0 0"/>
@@ -76,10 +77,10 @@
         </joint>
         <!-- Wheel transmissions -->
-        <transmission name="tran_${postfix}">
+        <transmission name="${prefix}_tran_${postfix}">
             <type>transmission_interface/SimpleTransmission</type>
-            <joint name="wheel_${postfix}_joint">
+            <joint name="${prefix}_wheel_${postfix}_joint">
                 <hardwareInterface>VelocityJointInterface</hardwareInterface>
             </joint>
-            <actuator name="motor_${postfix}">
+            <actuator name="${prefix}_motor_${postfix}">
                 <hardwareInterface>VelocityJointInterface</hardwareInterface>
                 <mechanicalReduction>1</mechanicalReduction>
@@ -93,8 +94,8 @@
     <!-- 3D Sensors -->
     <xacro:include filename="$(find tacbot_description)/urdf/kinect.xacro"/>
-    <sensor_kinect  parent="base_link"/>
-    <!-- Kobuki Gazebo simulation details  -->
+    <sensor_kinect prefix="${prefix}" parent="${prefix}_base_link"/>
+    <!-- Kobuki Gazebo simulation details   -->
     <xacro:include filename="$(find tacbot_description)/urdf/robot_gazebo.xacro"/>
-    <tacbot_sim/>
-    <tacbot_3dsensor_sim/>
+    <xacro:tacbot_sim prefix="${prefix}"/>
+    <tacbot_3dsensor_sim prefix="${prefix}"/>
 </robot>

File: tacbot_description/urdf/robot_gazebo.xacro (robot description, xacro)
@@ -2,6 +2,6 @@
 <robot name="tacbot_sim" xmlns:xacro="http://ros.org/wiki/xacro">
     <!-- Wheels macro -->
-    <xacro:macro name="wheel_sim" params="postfix">
-        <gazebo reference="wheel_${postfix}">
+    <xacro:macro name="wheel_sim" params="prefix postfix">
+        <gazebo reference="${prefix}_wheel_${postfix}">
             <mu1>1.0</mu1>
             <mu2>1.0</mu2>
@@ -12,9 +12,8 @@
             <material>Gazebo/Black</material>
         </gazebo>
-        <gazebo reference="wheel_${postfix}_joint"/>
     </xacro:macro>
-    <xacro:macro name="tacbot_sim">
+    <xacro:macro name="tacbot_sim" params="prefix">
         <!-- Base link -->
-        <gazebo reference="base_link">
+        <gazebo reference="${prefix}_base_link">
             <mu1>0.3</mu1>
             <mu2>0.3</mu2>
@@ -22,15 +21,15 @@
         </gazebo>
         <!-- Wheels -->
-        <xacro:wheel_sim postfix="FL"/>
-        <xacro:wheel_sim postfix="FR"/>
-        <xacro:wheel_sim postfix="BL"/>
-        <xacro:wheel_sim postfix="BR"/>
+        <xacro:wheel_sim prefix="${prefix}" postfix="FL"/>
+        <xacro:wheel_sim prefix="${prefix}" postfix="FR"/>
+        <xacro:wheel_sim prefix="${prefix}" postfix="BL"/>
+        <xacro:wheel_sim prefix="${prefix}" postfix="BR"/>
         <!-- Tacbot controller plugin for Gazebo -->
         <gazebo>
             <plugin name="tacbot_controller" filename="libgazebo_ros_tacbot.so">
-                <wheel_BL_joint_name>wheel_BL_joint</wheel_BL_joint_name>
-                <wheel_BR_joint_name>wheel_BR_joint</wheel_BR_joint_name>
-                <wheel_FL_joint_name>wheel_FL_joint</wheel_FL_joint_name>
-                <wheel_FR_joint_name>wheel_FR_joint</wheel_FR_joint_name>
+                <wheel_BL_joint_name>${prefix}_wheel_BL_joint</wheel_BL_joint_name>
+                <wheel_BR_joint_name>${prefix}_wheel_BR_joint</wheel_BR_joint_name>
+                <wheel_FL_joint_name>${prefix}_wheel_FL_joint</wheel_FL_joint_name>
+                <wheel_FR_joint_name>${prefix}_wheel_FR_joint</wheel_FR_joint_name>
                 <reg_kp>2.0</reg_kp>
                 <reg_ki>0</reg_ki>
@@ -45,6 +44,6 @@
     </xacro:macro>
     <!-- Microsoft Kinect for simulation -->
-    <xacro:macro name="tacbot_3dsensor_sim">
-        <gazebo reference="camera_link">
+    <xacro:macro name="tacbot_3dsensor_sim" params="prefix">
+        <gazebo reference="${prefix}_camera_link">
         <sensor type="depth" name="camera">
         <always_on>true</always_on>
@@ -63,13 +62,13 @@
         </camera>
         <plugin name="kinect_camera_controller" filename="libgazebo_ros_openni_kinect.so">
-            <cameraName>camera</cameraName>
+            <cameraName>kinect</cameraName>
             <alwaysOn>true</alwaysOn>
             <updateRate>10</updateRate>
-            <imageTopicName>rgb/image_raw</imageTopicName>
-            <depthImageTopicName>depth/image_raw</depthImageTopicName>
-            <pointCloudTopicName>depth/points</pointCloudTopicName>
-            <cameraInfoTopicName>rgb/camera_info</cameraInfoTopicName>
-            <depthImageCameraInfoTopicName>depth/camera_info</depthImageCameraInfoTopicName>
-            <frameName>camera_depth_optical_frame</frameName>
+            <imageTopicName>${prefix}/rgb/image_raw</imageTopicName>
+            <depthImageTopicName>${prefix}/depth/image_raw</depthImageTopicName>
+            <pointCloudTopicName>${prefix}/depth/points</pointCloudTopicName>
+            <cameraInfoTopicName>${prefix}/rgb/camera_info</cameraInfoTopicName>
+            <depthImageCameraInfoTopicName>${prefix}/depth/camera_info</depthImageCameraInfoTopicName>
+            <frameName>${prefix}_camera_depth_optical_frame</frameName>
             <baseline>0.1</baseline>
             <distortion_k1>0.0</distortion_k1>
