Commit message: Added Gazebo-ROS plugin for robot IMU sensor

File: tacbot_description/urdf/kinect.xacro (robot description, xacro)
@@ -1,63 +1,63 @@
 <?xml version="1.0"?>
 <robot name="sensor_kinect" xmlns:xacro="http://ros.org/wiki/xacro">
-  <xacro:property name="kinect_cam_py" value="-0.0125"/>
-        <xacro:property name="cam_px" value="0.085" />
-        <xacro:property name="cam_py" value="0.0125" />
-        <xacro:property name="cam_pz" value="0.14" />
+    <xacro:property name="kinect_cam_py" value="-0.0125"/>
+    <xacro:property name="cam_px" value="0.085" />
+    <xacro:property name="cam_py" value="0.0125" />
+    <xacro:property name="cam_pz" value="0.14" />
 	<xacro:property name="cam_or" value="0" />
 	<xacro:property name="cam_op" value="0" />
-        <xacro:property name="cam_oy" value="${pi}" />
-  <xacro:macro name="sensor_kinect" params="prefix parent">
+    <xacro:property name="cam_oy" value="${pi}" />
+    <xacro:macro name="sensor_kinect" params="prefix parent">
     <joint name="${prefix}_camera_rgb_joint" type="fixed">
-      <origin xyz="${cam_px} ${cam_py} ${cam_pz}" rpy="${cam_or} ${cam_op} ${cam_oy}"/>
-      <parent link="${parent}"/>
-      <child link="${prefix}_camera_rgb_frame" />
+        <origin xyz="${cam_px} ${cam_py} ${cam_pz}" rpy="${cam_or} ${cam_op} ${cam_oy}"/>
+        <parent link="${parent}"/>
+        <child link="${prefix}_camera_rgb_frame" />
     </joint>
     <link name="${prefix}_camera_rgb_frame"/>
     <joint name="${prefix}_camera_rgb_optical_joint" type="fixed">
-      <origin xyz="0 0 0" rpy="${-pi/2} 0 ${-pi/2}" />
-      <parent link="${prefix}_camera_rgb_frame" />
-      <child link="${prefix}_camera_rgb_optical_frame" />
+        <origin xyz="0 0 0" rpy="${-pi/2} 0 ${-pi/2}" />
+        <parent link="${prefix}_camera_rgb_frame" />
+        <child link="${prefix}_camera_rgb_optical_frame" />
     </joint>
     <link name="${prefix}_camera_rgb_optical_frame"/>
     <joint name="${prefix}_camera_joint" type="fixed">
-      <origin xyz="-0.031 ${-kinect_cam_py} -0.016" rpy="0 0 0"/>
-      <parent link="${prefix}_camera_rgb_frame"/>
-      <child link="${prefix}_camera_link"/>
+        <origin xyz="-0.031 ${-kinect_cam_py} -0.016" rpy="0 0 0"/>
+        <parent link="${prefix}_camera_rgb_frame"/>
+        <child link="${prefix}_camera_link"/>
     </joint>
-      <link name="${prefix}_camera_link">
-      <visual>
-       <origin xyz="0 0 0" rpy="0 0 ${pi/2}"/>
-        <geometry>
-         <mesh filename="package://turtlebot_description/meshes/sensors/kinect.dae"/>
-        </geometry>
-      </visual>
-  	  <collision>
-        <origin xyz="0.0 0.0 0.0" rpy="0 0 0"/>
-  	    <geometry>
-  	      <box size="0.07271 0.27794 0.073"/>
-  	    </geometry>
-  	  </collision>
-      <inertial>
-        <mass value="0.564" />
-        <origin xyz="0 0 0" />
-        <inertia ixx="0.003881243" ixy="0.0" ixz="0.0"
-                 iyy="0.000498940" iyz="0.0"
-                 izz="0.003879257" />
-      </inertial>
+    <link name="${prefix}_camera_link">
+        <visual>
+            <origin xyz="0 0 0" rpy="0 0 ${pi/2}"/>
+            <geometry>
+                <mesh filename="package://turtlebot_description/meshes/sensors/kinect.dae"/>
+            </geometry>
+        </visual>
+        <collision>
+            <origin xyz="0.0 0.0 0.0" rpy="0 0 0"/>
+            <geometry>
+                <box size="0.07271 0.27794 0.073"/>
+            </geometry>
+        </collision>
+        <inertial>
+            <mass value="0.564" />
+            <origin xyz="0 0 0" />
+            <inertia ixx="0.003881243" ixy="0.0" ixz="0.0"
+                     iyy="0.000498940" iyz="0.0"
+                     izz="0.003879257" />
+        </inertial>
     </link>
     <!-- For Gazebo simulation only -->
-	<joint name="${prefix}_camera_depth_joint" type="fixed">
-	  <origin xyz="0 ${2 * -kinect_cam_py} 0" rpy="0 0 0" />
-	  <parent link="${prefix}_camera_rgb_frame" />
-	  <child link="${prefix}_camera_depth_frame" />
-	</joint>
-	<link name="${prefix}_camera_depth_frame"/>
-	<joint name="${prefix}_camera_depth_optical_joint" type="fixed">
-	  <origin xyz="0 0 0" rpy="${-pi/2} 0 ${-pi/2}" />
-	  <parent link="${prefix}_camera_depth_frame" />
-	  <child link="${prefix}_camera_depth_optical_frame" />
-	</joint>
-	<link name="${prefix}_camera_depth_optical_frame"/>
-  </xacro:macro>
+    <joint name="${prefix}_camera_depth_joint" type="fixed">
+        <origin xyz="0 ${2 * -kinect_cam_py} 0" rpy="0 0 0" />
+        <parent link="${prefix}_camera_rgb_frame" />
+        <child link="${prefix}_camera_depth_frame" />
+    </joint>
+    <link name="${prefix}_camera_depth_frame"/>
+    <joint name="${prefix}_camera_depth_optical_joint" type="fixed">
+        <origin xyz="0 0 0" rpy="${-pi/2} 0 ${-pi/2}" />
+        <parent link="${prefix}_camera_depth_frame" />
+        <child link="${prefix}_camera_depth_optical_frame" />
+    </joint>
+    <link name="${prefix}_camera_depth_optical_frame"/>
+    </xacro:macro>
 </robot>

File: tacbot_description/urdf/robot.xacro (robot description, xacro)
@@ -92,4 +92,20 @@
     <xacro:wheel postfix="BL" side="-1" front="-1"/>
     <xacro:wheel postfix="BR" side="1" front="-1"/>
+    <!-- IMU sensor -->
+    <link name="${prefix}_imu_link">
+        <inertial>
+            <mass value="0.01"/>
+            <origin xyz="0 0 0" rpy="0 0 0"/>
+            <inertia ixx="0.0001" ixy="0" ixz="0"
+                     iyy="0.000001" iyz="0"
+                     izz="0.0001"/>
+        </inertial>
+    </link>
+    <joint name="${prefix}_imu_joint" type="fixed">
+        <axis xyz="0 1 0"/>
+        <origin xyz="0.05 0.0 0.1" rpy="0 0 0"/>
+        <parent link="${prefix}_base_link"/>
+        <child link="${prefix}_imu_link"/>
+    </joint>
     <!-- 3D Sensors -->
     <xacro:include filename="$(find tacbot_description)/urdf/kinect.xacro"/>
@@ -97,5 +113,6 @@
     <!-- Kobuki Gazebo simulation details   -->
     <xacro:include filename="$(find tacbot_description)/urdf/robot_gazebo.xacro"/>
-    <xacro:tacbot_sim prefix="${prefix}"/>
+    <tacbot_sim prefix="${prefix}"/>
+    <tacbot_imu_sim prefix="${prefix}"/>
     <tacbot_3dsensor_sim prefix="${prefix}"/>
 </robot>

File: tacbot_description/urdf/robot_gazebo.xacro (robot description, xacro)
@@ -33,6 +33,6 @@
                 <wheel_FR_joint_name>${prefix}_wheel_FR_joint</wheel_FR_joint_name>
                 <reg_kp>2.0</reg_kp>
-                <reg_ki>0</reg_ki>
-                <reg_kd>0</reg_kd>
+                <reg_ki>0.0</reg_ki>
+                <reg_kd>0.0</reg_kd>
                 <back_wheel_separation>.3</back_wheel_separation>
                 <front_wheel_separation>.3</front_wheel_separation>
@@ -41,4 +41,38 @@
                 <publish_tf>1</publish_tf>
             </plugin>
+        </gazebo>
+    </xacro:macro>
+    <!-- IMU sensor for simulation -->
+    <xacro:macro name="tacbot_imu_sim" params="prefix">
+        <gazebo reference="${prefix}_imu_link">
+        <sensor type="imu" name="${prefix}_imu">
+            <always_on>true</always_on>
+            <update_rate>100</update_rate>
+            <visualize>false</visualize>
+            <imu>
+                <noise>
+                    <type>gaussian</type>
+                    <rate>
+                        <mean>0.0</mean>
+                        <stddev>${0.0014*0.0014}</stddev>
+                        <bias_mean>0.0</bias_mean>
+                        <bias_stddev>0.0</bias_stddev>
+                    </rate>
+                    <accel>
+                        <mean>0.0</mean>
+                        <stddev>1.7e-2</stddev>
+                        <bias_mean>0.1</bias_mean>
+                        <bias_stddev>0.001</bias_stddev>
+                    </accel>
+                </noise>
+            </imu>
+        </sensor>
+        </gazebo>
+        <gazebo>
+        <plugin name="tacbot_imu" filename="libgazebo_tacbot_imu.so">
+            <imu_name>${prefix}_imu</imu_name>
+            <topic_name>imu_raw</topic_name>
+            <frame_name>imu_link</frame_name>
+        </plugin>
         </gazebo>
     </xacro:macro>
@@ -62,13 +96,13 @@
         </camera>
         <plugin name="kinect_camera_controller" filename="libgazebo_ros_openni_kinect.so">
-            <cameraName>kinect</cameraName>
+            <cameraName>${prefix}/kinect</cameraName>
             <alwaysOn>true</alwaysOn>
             <updateRate>10</updateRate>
-            <imageTopicName>${prefix}/rgb/image_raw</imageTopicName>
-            <depthImageTopicName>${prefix}/depth/image_raw</depthImageTopicName>
-            <pointCloudTopicName>${prefix}/depth/points</pointCloudTopicName>
-            <cameraInfoTopicName>${prefix}/rgb/camera_info</cameraInfoTopicName>
-            <depthImageCameraInfoTopicName>${prefix}/depth/camera_info</depthImageCameraInfoTopicName>
-            <frameName>${prefix}_camera_depth_optical_frame</frameName>
+            <imageTopicName>rgb/image_raw</imageTopicName>
+            <depthImageTopicName>depth/image_raw</depthImageTopicName>
+            <pointCloudTopicName>depth/points</pointCloudTopicName>
+            <cameraInfoTopicName>rgb/camera_info</cameraInfoTopicName>
+            <depthImageCameraInfoTopicName>depth/camera_info</depthImageCameraInfoTopicName>
+            <frameName>camera_depth_optical_frame</frameName>
             <baseline>0.1</baseline>
             <distortion_k1>0.0</distortion_k1>

Commit message: Navigation package configuration - step I

File: tacbot_description/urdf/kinect.xacro (robot description, xacro)
@@ -1,27 +1,8 @@
 <?xml version="1.0"?>
 <robot name="sensor_kinect" xmlns:xacro="http://ros.org/wiki/xacro">
-    <xacro:property name="kinect_cam_py" value="-0.0125"/>
-    <xacro:property name="cam_px" value="0.085" />
-    <xacro:property name="cam_py" value="0.0125" />
-    <xacro:property name="cam_pz" value="0.14" />
-	<xacro:property name="cam_or" value="0" />
-	<xacro:property name="cam_op" value="0" />
-    <xacro:property name="cam_oy" value="${pi}" />
-    <xacro:macro name="sensor_kinect" params="prefix parent">
-    <joint name="${prefix}_camera_rgb_joint" type="fixed">
-        <origin xyz="${cam_px} ${cam_py} ${cam_pz}" rpy="${cam_or} ${cam_op} ${cam_oy}"/>
+<xacro:macro name="sensor_kinect" params="prefix parent">
+    <joint name="${prefix}_camera_joint" type="fixed">
+        <origin xyz="0.085 0.0125 0.14" rpy="0 ${-pi/10} ${pi}"/>
         <parent link="${parent}"/>
-        <child link="${prefix}_camera_rgb_frame" />
-    </joint>
-    <link name="${prefix}_camera_rgb_frame"/>
-    <joint name="${prefix}_camera_rgb_optical_joint" type="fixed">
-        <origin xyz="0 0 0" rpy="${-pi/2} 0 ${-pi/2}" />
-        <parent link="${prefix}_camera_rgb_frame" />
-        <child link="${prefix}_camera_rgb_optical_frame" />
-    </joint>
-    <link name="${prefix}_camera_rgb_optical_frame"/>
-    <joint name="${prefix}_camera_joint" type="fixed">
-        <origin xyz="-0.031 ${-kinect_cam_py} -0.016" rpy="0 0 0"/>
-        <parent link="${prefix}_camera_rgb_frame"/>
         <child link="${prefix}_camera_link"/>
     </joint>
@@ -47,8 +28,20 @@
         </inertial>
     </link>
+    <joint name="${prefix}_camera_rgb_joint" type="fixed">
+        <origin xyz="0 -0.045 0" rpy="0 0 ${-pi}"/>
+        <parent link="${prefix}_camera_link"/>
+        <child link="${prefix}_camera_rgb_frame" />
+    </joint>
+    <link name="${prefix}_camera_rgb_frame"/>
+    <joint name="${prefix}_camera_rgb_optical_joint" type="fixed">
+        <origin xyz="0 0 0" rpy="${-pi/2} 0 ${-pi/2}" />
+        <parent link="${prefix}_camera_rgb_frame" />
+        <child link="${prefix}_camera_rgb_optical_frame" />
+    </joint>
+    <link name="${prefix}_camera_rgb_optical_frame"/>
     <!-- For Gazebo simulation only -->
     <joint name="${prefix}_camera_depth_joint" type="fixed">
-        <origin xyz="0 ${2 * -kinect_cam_py} 0" rpy="0 0 0" />
-        <parent link="${prefix}_camera_rgb_frame" />
+        <origin xyz="0 -0.02 0" rpy="0 0 ${-pi}" />
+        <parent link="${prefix}_camera_link" />
         <child link="${prefix}_camera_depth_frame" />
     </joint>
@@ -60,4 +53,4 @@
     </joint>
     <link name="${prefix}_camera_depth_optical_frame"/>
-    </xacro:macro>
+</xacro:macro>
 </robot>

File: tacbot_description/urdf/robot_gazebo.xacro (robot description, xacro)
@@ -91,6 +91,6 @@
             </image>
             <clip>
-                <near>0.05</near>
-                <far>8.0</far>
+                <near>0.4</near>
+                <far>6.0</far>
             </clip>
         </camera>
