Commit message: Update urdf model for Gazebo

File: tacbot_description/urdf/robot.xacro (robot description, xacro)
@@ -2,94 +2,106 @@
 <!-- Tacbot robot -->
 <robot name="tacbot" xmlns:xacro="http://www.ros.org/wiki/xacro">
-<!-- Constants-->
-<xacro:property name="base_length"  value=".35"/>
-<xacro:property name="base_width"   value=".3"/>
-<xacro:property name="base_height"  value=".055"/>
-<xacro:property name="wheel_width"  value=".04"/>
-<xacro:property name="wheel_radius" value=".06"/>
-<xacro:property name="wheel_dis"    value=".02"/>
-<!-- Base link definition-->
-<xacro:macro name="base_box"> <box size="${base_length} ${base_width} ${base_height}"/> </xacro:macro>
-<xacro:macro name="base_origin"> <origin xyz="0 0 ${wheel_radius}" rpy="0 0 0"/> </xacro:macro>
-<link name="base_link">
-    <visual>
-        <geometry>
-            <xacro:base_box/>
-        </geometry>
-        <xacro:base_origin/>
-        <material name="gray">
-		     <color rgba=".2 .2 .2 1" />
-        </material>
-    </visual>
-    <collision>
-        <geometry>
-            <xacro:base_box/>
-        </geometry>
-        <xacro:base_origin/>
-        <contact_coefficients mu="0" kp="1000.0" kd="1.0"/>
-    </collision>
-    <inertial>
-		  <origin xyz="0 0 0"/>
-        <mass value="3"/> <!-- 3 kg -->
-        <inertia ixx="0.3" ixy="0" ixz="0" iyy="0.3" iyz="0" izz="0.6" />
-    </inertial>
-</link>
-<xacro:macro name="wheel_cyl"> <cylinder radius="${wheel_radius}" length="${wheel_width}" /> </xacro:macro>
-<xacro:macro name="wheel_joint_origin">
-    <origin xyz="${front*(base_length/2-wheel_dis)} ${side*(base_width/2+wheel_width/2)} ${wheel_radius}" rpy="${pi/2} 0 0"/>
-</xacro:macro>
-<xacro:macro name="wheel" params="postfix side front">
-    <link name="wheel_${postfix}">
+    <!-- Constants-->
+    <xacro:property name="base_length"  value=".35"/>
+    <xacro:property name="base_width"   value=".3"/>
+    <xacro:property name="base_height"  value=".055"/>
+    <xacro:property name="wheel_width"  value=".04"/>
+    <xacro:property name="wheel_radius" value=".06"/>
+    <xacro:property name="wheel_dis"    value=".02"/>
+    <!-- Base dummy link -->
+    <link name="base_footprint"/>
+    <joint name="base_joint" type="fixed">
+      <origin xyz="0 0 0.0" rpy="0 0 0" />
+      <parent link="base_footprint"/>
+      <child link="base_link" />
+    </joint>
+    <!-- Base link definition-->
+    <xacro:macro name="base_box"> <box size="${base_length} ${base_width} ${base_height}"/> </xacro:macro>
+    <xacro:macro name="base_origin"> <origin xyz="0 0 ${wheel_radius}" rpy="0 0 0"/> </xacro:macro>
+    <link name="base_link">
         <visual>
             <geometry>
-		      	<xacro:wheel_cyl />
+                <xacro:base_box/>
             </geometry>
-				<origin xyz="0 0 0" rpy="0 0 0"/>
-            <material name="black">
-                <color rgba="0 0 0 1"/>
+            <xacro:base_origin/>
+            <material name="gray">
+                         <color rgba=".2 .2 .2 1" />
             </material>
         </visual>
         <collision>
             <geometry>
-                <xacro:wheel_cyl />
+                <xacro:base_box/>
             </geometry>
-				<origin xyz="0 0 0" rpy="0 0 0"/>
+            <xacro:base_origin/>
             <contact_coefficients mu="0" kp="1000.0" kd="1.0"/>
         </collision>
         <inertial>
-            <mass value="0.1" />
-            <inertia ixx="0.05" ixy="0.0" ixz="0.0" iyy="0.05" iyz="0.0" izz="0.05"/>
-    		</inertial>
+                      <origin xyz="0 0 0"/>
+            <mass value="3"/> <!-- 3 kg -->
+            <inertia ixx="0.3" ixy="0" ixz="0" iyy="0.3" iyz="0" izz="0.6" />
+        </inertial>
     </link>
-    <joint name="wheel_${postfix}_joint" type="continuous">
-        <parent link="base_link"/>
-        <child link="wheel_${postfix}"/>
-        <xacro:wheel_joint_origin />
-		  <axis xyz="0 0 1"/>
-        <dynamics damping="0" friction = "0" />
-        <limit effort="50" velocity="1.0" />
-        <safety_controller k_velocity="10" />
-    </joint>
-	 <transmission name="tran_${postfix}">
-        <type>transmission_interface/SimpleTransmission</type>
-    	  <joint name="wheel_${postfix}_joint">
-        	   <hardwareInterface>VelocityJointInterface</hardwareInterface>
+    <!-- Wheel macros -->
+    <xacro:macro name="wheel_cyl"> <cylinder radius="${wheel_radius}" length="${wheel_width}" /> </xacro:macro>
+    <xacro:macro name="wheel_joint_origin">
+        <origin xyz="${front*(base_length/2-wheel_dis)} ${side*(base_width/2+wheel_width/2)} ${wheel_radius}"
+                rpy="${pi/2} 0 0"/>
+    </xacro:macro>
+    <xacro:macro name="wheel" params="postfix side front">
+        <!-- Wheel links -->
+        <link name="wheel_${postfix}">
+            <visual>
+                <geometry>
+                    <xacro:wheel_cyl />
+                </geometry>
+                <origin xyz="0 0 0" rpy="0 0 0"/>
+                <material name="black">
+                    <color rgba="0 0 0 1"/>
+                </material>
+            </visual>
+            <collision>
+                <geometry>
+                    <xacro:wheel_cyl />
+                </geometry>
+                <origin xyz="0 0 0" rpy="0 0 0"/>
+                <contact_coefficients mu="0" kp="1000.0" kd="1.0"/>
+            </collision>
+            <inertial>
+                <mass value="0.1" />
+                <inertia ixx="0.05" ixy="0.0" ixz="0.0" iyy="0.05" iyz="0.0" izz="0.05"/>
+            </inertial>
+        </link>
+        <!-- Wheel joints -->
+        <joint name="wheel_${postfix}_joint" type="continuous">
+            <parent link="base_link"/>
+            <child link="wheel_${postfix}"/>
+            <xacro:wheel_joint_origin />
+            <axis xyz="0 0 1"/>
+            <dynamics damping="0" friction = "0" />
+            <limit effort="50" velocity="1.0" />
+            <safety_controller k_velocity="10" />
         </joint>
-    	  <actuator name="motor_${postfix}">
-        		<hardwareInterface>VelocityJointInterface</hardwareInterface>
-      		<mechanicalReduction>1</mechanicalReduction>
-    	  </actuator>
-  	 </transmission>
-</xacro:macro>
-<xacro:wheel postfix="FL" side="-1" front="1"/>
-<xacro:wheel postfix="FR" side="1" front="1"/>
-<xacro:wheel postfix="BL" side="-1" front="-1"/>
-<xacro:wheel postfix="BR" side="1" front="-1"/>
-<!-- 3D Sensors -->
-<xacro:include filename="$(find tacbot_description)/urdf/kinect.xacro"/>
-<sensor_kinect  parent="base_link"/>
-   <!-- Kobuki Gazebo simulation details  -->
-	<xacro:include filename="$(find tacbot_description)/urdf/robot_gazebo.xacro"/>
+        <!-- Wheel transmissions -->
+        <transmission name="tran_${postfix}">
+            <type>transmission_interface/SimpleTransmission</type>
+            <joint name="wheel_${postfix}_joint">
+                <hardwareInterface>VelocityJointInterface</hardwareInterface>
+            </joint>
+            <actuator name="motor_${postfix}">
+                <hardwareInterface>VelocityJointInterface</hardwareInterface>
+                <mechanicalReduction>1</mechanicalReduction>
+            </actuator>
+        </transmission>
+    </xacro:macro>
+    <xacro:wheel postfix="FL" side="-1" front="1"/>
+    <xacro:wheel postfix="FR" side="1" front="1"/>
+    <xacro:wheel postfix="BL" side="-1" front="-1"/>
+    <xacro:wheel postfix="BR" side="1" front="-1"/>
+    <!-- 3D Sensors -->
+    <xacro:include filename="$(find tacbot_description)/urdf/kinect.xacro"/>
+    <sensor_kinect  parent="base_link"/>
+    <!-- Kobuki Gazebo simulation details  -->
+    <xacro:include filename="$(find tacbot_description)/urdf/robot_gazebo.xacro"/>
     <tacbot_sim/>
-	<tacbot_3dsensor_sim/>
+    <tacbot_3dsensor_sim/>
 </robot>

File: tacbot_description/urdf/robot_gazebo.xacro (robot description, xacro)
@@ -1,138 +1,85 @@
 <?xml version="1.0"?>
 <robot name="tacbot_sim" xmlns:xacro="http://ros.org/wiki/xacro">
-	<!-- Base link -->
-	  <gazebo reference="base_link">
-	    <mu1>0.3</mu1>
-	    <mu2>0.3</mu2>
-	    <sensor type="contact" name="bumpers">
-	      <always_on>1</always_on>
-	      <update_rate>50.0</update_rate>
-	      <visualize>true</visualize>
-	      <contact>
-	        <collision>base_footprint_collision_base_link</collision>
-	      </contact>
-	    </sensor>
-		 <material>Gazebo/Grey</material>
-	  </gazebo>
-	<!-- Wheels -->
-	<xacro:macro name="wheel_sim" params="postfix">
-    <gazebo reference="wheel_${postfix}">
-	    <mu1>1.0</mu1>
-	    <mu2>1.0</mu2>
-	    <kp>1000000.0</kp>
-	    <kd>100.0</kd>
-	    <minDepth>0.001</minDepth>
-	    <maxVel>1.0</maxVel>
-		 <material>Gazebo/Black</material>
-    </gazebo>
-    <gazebo reference="wheel_${postfix}_joint">
-    </gazebo>
-	</xacro:macro>
-<xacro:wheel_sim postfix="FL"/>
-<xacro:wheel_sim postfix="FR"/>
-<xacro:wheel_sim postfix="BL"/>
-<xacro:wheel_sim postfix="BR"/>
-<!--	  <gazebo reference="cliff_sensor_front_link">
-	    <sensor type="ray" name="cliff_sensor_front">
-	      <always_on>true</always_on>
-	      <update_rate>50</update_rate>
-	      <visualize>true</visualize>
-	      <ray>
-	        <scan>
-	          <horizontal>
-	            <samples>50</samples>
-	            <resolution>1.0</resolution>
-	            <min_angle>-0.0436</min_angle>
-	            <max_angle>0.0436</max_angle>
-	          </horizontal>
-	        </scan>
-	        <range>
-	          <min>0.01</min>
-	          <max>0.15</max>
-	          <resolution>1.0</resolution>
-	        </range>
-	      </ray>
-	    </sensor>
-	  </gazebo>-->
-	 <gazebo reference="imu_link">
-	   <sensor type="imu" name="imu">
-        <always_on>true</always_on>
-        <update_rate>50</update_rate>
-        <visualize>false</visualize>
-        <imu>
-          <noise>
-            <type>gaussian</type>
-	          <rate>
-	            <mean>0.0</mean>
-	            <stddev>${0.0014*0.0014}</stddev> <!-- 0.25 x 0.25 (deg/s) -->
-	            <bias_mean>0.0</bias_mean>
-	            <bias_stddev>0.0</bias_stddev>
-	          </rate>
-		        <accel>
-			        <mean>0.0</mean>
-			        <stddev>1.7e-2</stddev>
-			        <bias_mean>0.1</bias_mean>
-			        <bias_stddev>0.001</bias_stddev>
-		        </accel>
-          </noise>
-	      </imu>
-      </sensor>
-	  </gazebo>
-  <!-- Microsoft Kinect for simulation -->
-  <xacro:macro name="tacbot_3dsensor_sim">
-    <gazebo reference="camera_link">
-      <sensor type="depth" name="camera">
+    <!-- Wheels macro -->
+    <xacro:macro name="wheel_sim" params="postfix">
+        <gazebo reference="wheel_${postfix}">
+            <mu1>1.0</mu1>
+            <mu2>1.0</mu2>
+            <kp>10000.0</kp>
+            <kd>10.0</kd>
+            <minDepth>0.001</minDepth>
+            <maxVel>1.0</maxVel>
+            <material>Gazebo/Black</material>
+        </gazebo>
+        <gazebo reference="wheel_${postfix}_joint"/>
+    </xacro:macro>
+    <xacro:macro name="tacbot_sim">
+        <!-- Base link -->
+        <gazebo reference="base_link">
+            <mu1>0.3</mu1>
+            <mu2>0.3</mu2>
+            <material>Gazebo/Grey</material>
+        </gazebo>
+        <!-- Wheels -->
+        <xacro:wheel_sim postfix="FL"/>
+        <xacro:wheel_sim postfix="FR"/>
+        <xacro:wheel_sim postfix="BL"/>
+        <xacro:wheel_sim postfix="BR"/>
+        <!-- Tacbot controller plugin for Gazebo -->
+        <gazebo>
+            <plugin name="tacbot_controller" filename="libgazebo_ros_tacbot.so">
+                <wheel_BL_joint_name>wheel_BL_joint</wheel_BL_joint_name>
+                <wheel_BR_joint_name>wheel_BR_joint</wheel_BR_joint_name>
+                <wheel_FL_joint_name>wheel_FL_joint</wheel_FL_joint_name>
+                <wheel_FR_joint_name>wheel_FR_joint</wheel_FR_joint_name>
+                <reg_kp>1.0</reg_kp>
+                <reg_ki>0</reg_ki>
+                <reg_kd>0</reg_kd>
+                <back_wheel_separation>.3</back_wheel_separation>
+                <front_wheel_separation>.3</front_wheel_separation>
+                <wheel_diameter>0.11</wheel_diameter>
+                <max_torque>0.5</max_torque>
+                <publish_tf>1</publish_tf>
+            </plugin>
+        </gazebo>
+    </xacro:macro>
+    <!-- Microsoft Kinect for simulation -->
+    <xacro:macro name="tacbot_3dsensor_sim">
+        <gazebo reference="camera_link">
+        <sensor type="depth" name="camera">
         <always_on>true</always_on>
         <update_rate>20.0</update_rate>
         <camera>
-          <horizontal_fov>${60.0*pi/180.0}</horizontal_fov>
-          <image>
-            <format>R8G8B8</format>
-            <width>640</width>
-            <height>480</height>
-          </image>
-          <clip>
-            <near>0.05</near>
-            <far>8.0</far>
-          </clip>
+            <horizontal_fov>${60.0*pi/180.0}</horizontal_fov>
+            <image>
+                <format>R8G8B8</format>
+                <width>640</width>
+                <height>480</height>
+            </image>
+            <clip>
+                <near>0.05</near>
+                <far>8.0</far>
+            </clip>
         </camera>
         <plugin name="kinect_camera_controller" filename="libgazebo_ros_openni_kinect.so">
-          <cameraName>camera</cameraName>
-          <alwaysOn>true</alwaysOn>
-          <updateRate>10</updateRate>
-          <imageTopicName>rgb/image_raw</imageTopicName>
-          <depthImageTopicName>depth/image_raw</depthImageTopicName>
-          <pointCloudTopicName>depth/points</pointCloudTopicName>
-          <cameraInfoTopicName>rgb/camera_info</cameraInfoTopicName>
-          <depthImageCameraInfoTopicName>depth/camera_info</depthImageCameraInfoTopicName>
-          <frameName>camera_depth_optical_frame</frameName>
-          <baseline>0.1</baseline>
-          <distortion_k1>0.0</distortion_k1>
-          <distortion_k2>0.0</distortion_k2>
-          <distortion_k3>0.0</distortion_k3>
-          <distortion_t1>0.0</distortion_t1>
-          <distortion_t2>0.0</distortion_t2>
-          <pointCloudCutoff>0.4</pointCloudCutoff>
+            <cameraName>camera</cameraName>
+            <alwaysOn>true</alwaysOn>
+            <updateRate>10</updateRate>
+            <imageTopicName>rgb/image_raw</imageTopicName>
+            <depthImageTopicName>depth/image_raw</depthImageTopicName>
+            <pointCloudTopicName>depth/points</pointCloudTopicName>
+            <cameraInfoTopicName>rgb/camera_info</cameraInfoTopicName>
+            <depthImageCameraInfoTopicName>depth/camera_info</depthImageCameraInfoTopicName>
+            <frameName>camera_depth_optical_frame</frameName>
+            <baseline>0.1</baseline>
+            <distortion_k1>0.0</distortion_k1>
+            <distortion_k2>0.0</distortion_k2>
+            <distortion_k3>0.0</distortion_k3>
+            <distortion_t1>0.0</distortion_t1>
+            <distortion_t2>0.0</distortion_t2>
+            <pointCloudCutoff>0.4</pointCloudCutoff>
         </plugin>
-      </sensor>
-    </gazebo>
-  </xacro:macro>
-<!--<gazebo>
-  <plugin name="gazebo_ros_control" filename="libgazebo_ros_control.so">
-    <robotNamespace>/tacbot</robotNamespace>
-  </plugin>
-</gazebo> -->
-<gazebo>
-	    <plugin name="kobuki_controller" filename="libgazebo_ros_kobuki.so">
-	      <publish_tf>1</publish_tf>
-	      <left_wheel_joint_name>wheel_left_joint</left_wheel_joint_name>
-	      <right_wheel_joint_name>wheel_right_joint</right_wheel_joint_name>
-	      <wheel_separation>.230</wheel_separation>
-	      <wheel_diameter>0.070</wheel_diameter>
-	      <torque>1.0</torque>
-	      <velocity_command_timeout>0.6</velocity_command_timeout>
-        <imu_name>imu</imu_name>
-	    </plugin>
-	  </gazebo>
+        </sensor>
+        </gazebo>
   </xacro:macro>
 </robot>

Commit message: Added licence Cleaned code and topic names

File: tacbot_description/urdf/robot.xacro (robot description, xacro)
@@ -3,5 +3,5 @@
 <robot name="tacbot" xmlns:xacro="http://ros.org/wiki/xacro">
     <!-- Constants-->
-	 <xacro:property name="prefix"		 value="r1"/>
+	<xacro:property name="prefix"		value="$(arg prefix)"/>
     <xacro:property name="base_length"  value=".297"/>
     <xacro:property name="base_width"   value=".189"/>

File: tacbot_description/urdf/robot_gazebo.xacro (robot description, xacro)
@@ -96,5 +96,5 @@
         </camera>
         <plugin name="kinect_camera_controller" filename="libgazebo_ros_openni_kinect.so">
-            <cameraName>${prefix}/kinect</cameraName>
+            <cameraName>kinect</cameraName>
             <alwaysOn>true</alwaysOn>
             <updateRate>10</updateRate>
