Commit message: Updated urdf model of robot. Added laser scanner

File: tacbot_description/urdf/robot.xacro (robot description, xacro)
@@ -2,117 +2,37 @@
 <!-- Tacbot robot -->
 <robot name="tacbot" xmlns:xacro="http://ros.org/wiki/xacro">
-    <!-- Constants-->
-	<xacro:property name="prefix"		value="$(arg prefix)"/>
-    <xacro:property name="base_length"  value=".297"/>
-    <xacro:property name="base_width"   value=".189"/>
-    <xacro:property name="base_height"  value=".06"/>
-    <xacro:property name="wheel_width"  value=".055"/>
-    <xacro:property name="wheel_radius" value=".055"/>
-    <xacro:property name="wheel_dis"    value=".0235"/>
-    <!-- Base dummy link -->
-    <link name="${prefix}_base_footprint"/>
-    <joint name="${prefix}_base_joint" type="fixed">
-      <origin xyz="0 0 0.0" rpy="0 0 0" />
-      <parent link="${prefix}_base_footprint"/>
-      <child link="${prefix}_base_link" />
-    </joint>
-    <!-- Base link definition-->
-    <xacro:macro name="base_box"> <box size="${base_length} ${base_width} ${base_height}"/> </xacro:macro>
-    <xacro:macro name="base_origin"> <origin xyz="0 0 ${wheel_radius}" rpy="0 0 0"/> </xacro:macro>
-    <link name="${prefix}_base_link">
-        <visual>
-            <geometry>
-                <xacro:base_box/>
-            </geometry>
-            <xacro:base_origin/>
-            <material name="gray">
-                <color rgba=".2 .2 .2 1" />
-            </material>
-        </visual>
-        <collision>
-            <geometry>
-                <xacro:base_box/>
-            </geometry>
-            <xacro:base_origin/>
-        </collision>
-        <inertial>
-            <mass value="4"/> <!-- 4 kg -->
-            <origin xyz="0 0 0"/>
-            <inertia ixx="0.02" ixy="0" ixz="0" iyy="0.02" iyz="0" izz="0.03" />
-        </inertial>
-    </link>
-    <!-- Wheel links -->
-    <xacro:macro name="wheel" params="postfix side front">
-        <link name="${prefix}_wheel_${postfix}">
-            <visual>
-                <geometry>
-                    <cylinder radius="${wheel_radius}" length="${wheel_width}"/>
-                </geometry>
-                <origin xyz="0 0 0" rpy="0 0 0"/>
-                <material name="black">
-                    <color rgba="0 0 0 1"/>
-                </material>
-            </visual>
-            <collision>
-                <geometry>
-                    <cylinder radius="${wheel_radius}" length="${wheel_width}"/>
-                </geometry>
-                <origin xyz="0 0 0" rpy="0 0 0"/>
-            </collision>
-            <inertial>
-                <mass value="0.2" />
-                <inertia ixx="0.005" ixy="0.0" ixz="0.0" iyy="0.005" iyz="0.0" izz="0.005"/>
-            </inertial>
-        </link>
-        <!-- Wheel joints -->
-        <joint name="${prefix}_wheel_${postfix}_joint" type="continuous">
-            <parent link="${prefix}_base_link"/>
-            <child link="${prefix}_wheel_${postfix}"/>
-            <origin xyz="${front*(base_length/2-wheel_dis)} ${side*(base_width/2+wheel_width/2)} ${wheel_radius}"
-                    rpy="${pi/2} 0 0"/>
-            <axis xyz="0 0 1"/>
-            <dynamics damping="0" friction = "0" />
-            <limit effort="5" velocity="1.0" />
-            <safety_controller k_velocity="5" />
-        </joint>
-        <!-- Wheel transmissions -->
-        <transmission name="${prefix}_tran_${postfix}">
-            <type>transmission_interface/SimpleTransmission</type>
-            <joint name="${prefix}_wheel_${postfix}_joint">
-                <hardwareInterface>VelocityJointInterface</hardwareInterface>
-            </joint>
-            <actuator name="${prefix}_motor_${postfix}">
-                <hardwareInterface>VelocityJointInterface</hardwareInterface>
-                <mechanicalReduction>1</mechanicalReduction>
-            </actuator>
-        </transmission>
-    </xacro:macro>
-    <xacro:wheel postfix="FL" side="-1" front="1"/>
-    <xacro:wheel postfix="FR" side="1" front="1"/>
-    <xacro:wheel postfix="BL" side="-1" front="-1"/>
-    <xacro:wheel postfix="BR" side="1" front="-1"/>
+    <!-- Properties -->
+	<xacro:property name="prefix" value="$(arg prefix)"/>
+    <xacro:include filename="utils.xacro"/>
+    <xacro:include filename="materials.xacro"/>
+    <!-- Base link and wheels -->
+    <xacro:include filename="base.xacro"/>
+    <xacro:include filename="base.gazebo.xacro"/>
+    <xacro:include filename="wheel.xacro"/>
+    <xacro:include filename="wheel.gazebo.xacro"/>
+    <base_link prefix="${prefix}"/>
+    <base_gazebo prefix="${prefix}"/>
+    <wheel prefix="${prefix}" postfix="FL" side="-1" front="1"/>
+    <wheel prefix="${prefix}" postfix="FR" side="1"  front="1"/>
+    <wheel prefix="${prefix}" postfix="BL" side="-1" front="-1"/>
+    <wheel prefix="${prefix}" postfix="BR" side="1"  front="-1"/>
+    <wheel_gazebo prefix="${prefix}" postfix="FL"/>
+    <wheel_gazebo prefix="${prefix}" postfix="FR"/>
+    <wheel_gazebo prefix="${prefix}" postfix="BL"/>
+    <wheel_gazebo prefix="${prefix}" postfix="BR"/>
     <!-- IMU sensor -->
-    <link name="${prefix}_imu_link">
-        <inertial>
-            <mass value="0.01"/>
-            <origin xyz="0 0 0" rpy="0 0 0"/>
-            <inertia ixx="0.0001" ixy="0" ixz="0"
-                     iyy="0.000001" iyz="0"
-                     izz="0.0001"/>
-        </inertial>
-    </link>
-    <joint name="${prefix}_imu_joint" type="fixed">
-        <axis xyz="0 1 0"/>
-        <origin xyz="0.05 0.0 0.1" rpy="0 0 0"/>
-        <parent link="${prefix}_base_link"/>
-        <child link="${prefix}_imu_link"/>
-    </joint>
-    <!-- 3D Sensors -->
-    <xacro:include filename="$(find tacbot_description)/urdf/kinect.xacro"/>
+    <xacro:include filename="sensors/imu.xacro"/>
+    <xacro:include filename="sensors/imu.gazebo.xacro"/>
+    <sensor_imu prefix="${prefix}" parent="${prefix}_base_link"/>
+    <sensor_imu_gazebo prefix="${prefix}"/>
+    <!-- Kinect sensor -->
+    <xacro:include filename="sensors/kinect.xacro"/>
+    <xacro:include filename="sensors/kinect.gazebo.xacro"/>
     <sensor_kinect prefix="${prefix}" parent="${prefix}_base_link"/>
-    <!-- Kobuki Gazebo simulation details   -->
-    <xacro:include filename="$(find tacbot_description)/urdf/robot_gazebo.xacro"/>
-    <tacbot_sim prefix="${prefix}"/>
-    <tacbot_imu_sim prefix="${prefix}"/>
-    <tacbot_3dsensor_sim prefix="${prefix}"/>
+    <sensor_kinect_gazebo prefix="${prefix}"/>
+    <!-- Hokuyo LX30 -->
+    <xacro:include filename="sensors/hokuyo_lx30.xacro"/>
+    <xacro:include filename="sensors/hokuyo_lx30.gazebo.xacro"/>
+    <hokuyo_lx30 prefix="${prefix}" parent="${prefix}_base_link"/>
+    <hokuyo_lx30_gazebo prefix="${prefix}"/>
 </robot>

File: tacbot_description/urdf/sensors/kinect.xacro (robot description, xacro)
@@ -3,5 +3,5 @@
 <xacro:macro name="sensor_kinect" params="prefix parent">
     <joint name="${prefix}_camera_joint" type="fixed">
-        <origin xyz="0.085 0.0125 0.14" rpy="0 ${-pi/10} ${pi}"/>
+        <origin xyz="-0.1 0.0 0.2" rpy="0 0 0"/>
         <parent link="${parent}"/>
         <child link="${prefix}_camera_link"/>
@@ -29,5 +29,5 @@
     </link>
     <joint name="${prefix}_camera_rgb_joint" type="fixed">
-        <origin xyz="0 -0.045 0" rpy="0 0 ${-pi}"/>
+        <origin xyz="0 -0.045 0" rpy="0 0 0"/>
         <parent link="${prefix}_camera_link"/>
         <child link="${prefix}_camera_rgb_frame" />
@@ -40,7 +40,6 @@
     </joint>
     <link name="${prefix}_camera_rgb_optical_frame"/>
-    <!-- For Gazebo simulation only -->
     <joint name="${prefix}_camera_depth_joint" type="fixed">
-        <origin xyz="0 -0.02 0" rpy="0 0 ${-pi}" />
+        <origin xyz="0 -0.02 0" rpy="0 0 0" />
         <parent link="${prefix}_camera_link" />
         <child link="${prefix}_camera_depth_frame" />
