Commit message: Refactoring of robot urdf model Corrected robot drive gazebo plugin and configured sensors

File: tacbot_description/urdf/base.gazebo.xacro (robot description, xacro)
@@ -6,4 +6,9 @@
             <mu1>0.3</mu1>
             <mu2>0.3</mu2>
+            <gravity>true</gravity>
+            <material>Gazebo/Grey</material>
+        </gazebo>
+        <!-- Kinect mounting -->
+        <gazebo reference="${prefix}_kinect_mounting">
             <material>Gazebo/Grey</material>
         </gazebo>
@@ -11,9 +16,9 @@
         <gazebo>
             <plugin name="tacbot_controller" filename="libgazebo_ros_tacbot.so">
-                <wheel_BL_joint_name>${prefix}_wheel_BL_joint</wheel_BL_joint_name>
-                <wheel_BR_joint_name>${prefix}_wheel_BR_joint</wheel_BR_joint_name>
-                <wheel_FL_joint_name>${prefix}_wheel_FL_joint</wheel_FL_joint_name>
-                <wheel_FR_joint_name>${prefix}_wheel_FR_joint</wheel_FR_joint_name>
-                <reg_kp>2.0</reg_kp>
+                <wheel_BL_joint>${prefix}_wheel_BL_joint</wheel_BL_joint>
+                <wheel_BR_joint>${prefix}_wheel_BR_joint</wheel_BR_joint>
+                <wheel_FL_joint>${prefix}_wheel_FL_joint</wheel_FL_joint>
+                <wheel_FR_joint>${prefix}_wheel_FR_joint</wheel_FR_joint>
+                <reg_kp>1.0</reg_kp>
                 <reg_ki>0.0</reg_ki>
                 <reg_kd>0.0</reg_kd>

File: tacbot_description/urdf/base.xacro (robot description, xacro)
@@ -10,5 +10,5 @@
         <link name="${prefix}_base_footprint"/>
         <joint name="${prefix}_base_joint" type="fixed">
-            <origin xyz="0 0 5" rpy="0 0 0" />
+            <origin xyz="0 0 ${wheel_radius+base_height/2}" rpy="0 0 0" />
             <parent link="${prefix}_base_footprint"/>
             <child link="${prefix}_base_link"/>
@@ -29,6 +29,6 @@
             </collision>
             <inertial>
+                <origin xyz="0 0 0" rpy="0 0 0"/>
                 <mass value="${base_mass}"/>
-                <origin xyz="0 0 0"/>
                 <cuboid_inertia m="${base_mass}" x="${base_length}" y="${base_width}" z="${base_height}"/>
             </inertial>
@@ -38,4 +38,5 @@
         <xacro:property name="kinect_mounting_y" value="0.06"/>
         <xacro:property name="kinect_mounting_z" value="0.15"/>
+        <xacro:property name="kinect_mounting_mass" value="0.2"/>
         <joint name="${prefix}_kinect_mounting_joint" type="fixed">
             <origin xyz="-0.1 0 ${base_height/2 + kinect_mounting_z/2}" rpy="0 0 0" />
@@ -60,5 +61,5 @@
                 <mass value="0.2"/>
                 <origin xyz="0 0 0"/>
-                <cuboid_inertia m="0.2" x="${kinect_mounting_x}" y="${kinect_mounting_y}" z="${kinect_mounting_z}"/>
+                <cuboid_inertia m="${kinect_mounting_mass}" x="${kinect_mounting_x}" y="${kinect_mounting_y}" z="${kinect_mounting_z}"/>
             </inertial>
         </link>

File: tacbot_description/urdf/robot.xacro (robot description, xacro)
@@ -4,17 +4,18 @@
     <!-- Properties -->
 	<xacro:property name="prefix" value="$(arg prefix)"/>
+	<xacro:arg name="prefix" default="r1"/>
     <xacro:include filename="utils.xacro"/>
     <xacro:include filename="materials.xacro"/>
     <!-- Base link and wheels -->
     <xacro:include filename="base.xacro"/>
+    <xacro:include filename="wheel.xacro"/>
+    <base_link prefix="${prefix}"/>
+    <wheel prefix="${prefix}" postfix="FL" side="1" front="1"/>
+    <wheel prefix="${prefix}" postfix="FR" side="-1"  front="1"/>
+    <wheel prefix="${prefix}" postfix="BL" side="1" front="-1"/>
+    <wheel prefix="${prefix}" postfix="BR" side="-1"  front="-1"/>
     <xacro:include filename="base.gazebo.xacro"/>
-    <xacro:include filename="wheel.xacro"/>
+    <base_gazebo prefix="${prefix}"/>
     <xacro:include filename="wheel.gazebo.xacro"/>
-    <base_link prefix="${prefix}"/>
-    <base_gazebo prefix="${prefix}"/>
-    <wheel prefix="${prefix}" postfix="FL" side="-1" front="1"/>
-    <wheel prefix="${prefix}" postfix="FR" side="1"  front="1"/>
-    <wheel prefix="${prefix}" postfix="BL" side="-1" front="-1"/>
-    <wheel prefix="${prefix}" postfix="BR" side="1"  front="-1"/>
     <wheel_gazebo prefix="${prefix}" postfix="FL"/>
     <wheel_gazebo prefix="${prefix}" postfix="FR"/>

File: tacbot_description/urdf/sensors/hokuyo_lx30.gazebo.xacro (robot description, xacro)
@@ -4,34 +4,32 @@
     <xacro:property name="max_angle" value=""/>
     <xacro:macro name="hokuyo_lx30_gazebo" params="prefix">
-        <gazebo reference="${prefix}_hokuyo_link">
-        <sensor type="gpu_ray" name="hokuyo">
-          <always_on>true</always_on>
-          <update_rate>20</update_rate>
-          <pose>0 0 0 0 0 0</pose>
-          <visualize>true</visualize>
-          <ray>
-            <scan>
-              <horizontal>
-                <samples>640</samples>
-                <resolution>1</resolution>
-                <min_angle>-1.570796</min_angle>
-                <max_angle>1.570796</max_angle>
-              </horizontal>
-            </scan>
-            <range>
-              <min>0.08</min>
-              <max>10.0</max>
-              <resolution>0.01</resolution>
-            </range>
-          </ray>
-          <plugin name="gazebo_ros_laser_controller" filename="libgazebo_ros_gpu_laser.so">
-            <gaussianNoise>0.005</gaussianNoise>
-            <alwaysOn>true</alwaysOn>
-            <updateRate>20</updateRate>
-            <topicName>${prefix}_scan</topicName>
-            <frameName>${prefix}_hokuyo_link</frameName>
-            <hokuyoMinIntensity>101</hokuyoMinIntensity>
-          </plugin>
-        </sensor>
+        <gazebo reference="${prefix}/hokuyo_link">
+            <material>Gazebo/Black</material>
+            <sensor type="ray" name="hokuyo">
+                <always_on>true</always_on>
+                <update_rate>20</update_rate>
+                <pose>0 0 0 0 0 0</pose>
+                <visualize>false</visualize>
+                <ray>
+                    <scan>
+                        <horizontal>
+                            <samples>640</samples>
+                            <resolution>1</resolution>
+                            <min_angle>-1.570796</min_angle>
+                            <max_angle>1.570796</max_angle>
+                        </horizontal>
+                    </scan>
+                    <range>
+                        <min>0.08</min>
+                        <max>10.0</max>
+                        <resolution>0.01</resolution>
+                    </range>
+                </ray>
+                <plugin name="gazebo_ros_laser_controller" filename="libgazebo_ros_laser.so">
+                    <topicName>scan</topicName>
+                    <frameName>hokuyo_link</frameName>
+                    <robotNamespace>${prefix}</robotNamespace>
+                </plugin>
+            </sensor>
         </gazebo>
     </xacro:macro>

File: tacbot_description/urdf/sensors/hokuyo_lx30.xacro (robot description, xacro)
@@ -6,11 +6,10 @@
         <xacro:property name="hokuyo_z" value="0.06"/>
         <xacro:property name="hokuyo_mass" value="0.1"/>
-        <joint name="${prefix}_hokuyo_joint" type="fixed">
-            <axis xyz="0 1 0" />
+        <joint name="${prefix}/hokuyo_joint" type="fixed">
             <origin xyz="0.12 0.0 ${hokuyo_z/2 + base_height/2}" rpy="0 0 0"/>
             <parent link="${parent}"/>
-            <child link="${prefix}_hokuyo_link"/>
+            <child link="${prefix}/hokuyo_link"/>
         </joint>
-        <link name="${prefix}_hokuyo_link" type="laser">
+        <link name="${prefix}/hokuyo_link" type="laser">
             <visual>
                 <origin xyz="0 0 0" rpy="0 0 0"/>

File: tacbot_description/urdf/utils.xacro (robot description, xacro)
@@ -1,15 +1,15 @@
 <?xml version="1.0"?>
 <robot xmlns:xacro="http://ros.org/wiki/xacro">
-        <!--Inertia of the cuboid in kg*m^2-->
-        <xacro:macro name="cuboid_inertia" params="m x y z">
-          <inertia  ixx="${m*(y*y+z*z)/12}" ixy = "0" ixz = "0"
-                    iyy="${m*(x*x+z*z)/12}" iyz = "0"
-                    izz="${m*(x*x+z*z)/12}" />
-        </xacro:macro>
-        <!--Inertia of the cylinder in kg*m^2-->
-        <xacro:macro name="cylinder_inertia" params="m r h">
-          <inertia  ixx="${m*(3*r*r+h*h)/12}" ixy = "0" ixz = "0"
-                    iyy="${m*(3*r*r+h*h)/12}" iyz = "0"
-                    izz="${m*(r*r)/2}" />
-        </xacro:macro>
+    <!--Inertia of the cuboid in kg*m^2-->
+    <xacro:macro name="cuboid_inertia" params="m:=1.0 x y z">
+      <inertia  ixx="${m*(y*y+z*z)/12.0}" ixy = "0.0" ixz = "0.0"
+                iyy="${m*(x*x+z*z)/12.0}" iyz = "0.0"
+                izz="${m*(x*x+z*z)/12.0}" />
+    </xacro:macro>
+    <!--Inertia of the cylinder in kg*m^2-->
+    <xacro:macro name="cylinder_inertia" params="m:=1.0 r h">
+      <inertia  ixx="${m*(3*r*r+h*h)/12.0}" ixy = "0.0" ixz = "0.0"
+                iyy="${m*(3*r*r+h*h)/12.0}" iyz = "0.0"
+                izz="${m*(r*r)/2.0}" />
+    </xacro:macro>
 </robot>

File: tacbot_description/urdf/wheel.gazebo.xacro (robot description, xacro)
@@ -5,8 +5,8 @@
             <mu1>1.0</mu1>
             <mu2>1.0</mu2>
-            <kp>100000.0</kp>
-            <kd>10.0</kd>
             <minDepth>0.001</minDepth>
-            <maxVel>1.0</maxVel>
+            <maxVel>10</maxVel>
+            <kp>1000000.0</kp>
+            <kd>1.0</kd>
             <material>Gazebo/Black</material>
         </gazebo>

File: tacbot_description/urdf/wheel.xacro (robot description, xacro)
@@ -4,6 +4,6 @@
     <xacro:property name="wheel_width"  value=".055"/>
     <xacro:property name="wheel_radius" value=".055"/>
-    <xacro:property name="wheel_dis"    value=".0235"/>
-    <xacro:property name="wheel_mass"   value=".2"/>
+    <xacro:property name="wheel_dis"    value=".024"/>
+    <xacro:property name="wheel_mass"   value=".5"/>
     <xacro:macro name="wheel" params="prefix postfix side front">
         <!-- Wheel joints -->
@@ -11,10 +11,7 @@
             <parent link="${prefix}_base_link"/>
             <child link="${prefix}_wheel_${postfix}"/>
-            <origin xyz="${front*(base_length/2-wheel_dis)} ${side*(base_width/2+wheel_width/2)} 0"
-                    rpy="${pi/2} 0 0"/>
+            <origin xyz="${front*(base_length/2-wheel_dis)} ${side*(base_width/2+wheel_width/2 + 0.005)} 0"
+                    rpy="${-pi/2} 0 0"/>
             <axis xyz="0 0 1"/>
-            <dynamics damping="0" friction = "0" />
-            <limit effort="5" velocity="1.0" />
-            <safety_controller k_velocity="5" />
         </joint>
         <!-- Wheel links -->
@@ -34,4 +31,5 @@
             </collision>
             <inertial>
+                <origin xyz="0 0 0" rpy="0 0 0"/>
                 <mass value="${wheel_mass}" />
                 <cylinder_inertia m="${wheel_mass}" r="${wheel_radius}" h="${wheel_width}"/>

Commit message: Configurations cleaning Removed base_footprint from model

File: tacbot_description/urdf/base.gazebo.xacro (robot description, xacro)
@@ -27,5 +27,5 @@
                 <wheel_diameter>0.11</wheel_diameter>
                 <max_torque>0.4</max_torque>
-                <publish_tf>1</publish_tf>
+                <publish_tf>false</publish_tf>
             </plugin>
         </gazebo>

File: tacbot_description/urdf/base.xacro (robot description, xacro)
@@ -7,11 +7,4 @@
     <xacro:property name="base_mass"    value="4"/>
     <xacro:macro name="base_link" params="prefix">
-        <!-- Base footprint -->
-        <link name="${prefix}_base_footprint"/>
-        <joint name="${prefix}_base_joint" type="fixed">
-            <origin xyz="0 0 ${wheel_radius+base_height/2}" rpy="0 0 0" />
-            <parent link="${prefix}_base_footprint"/>
-            <child link="${prefix}_base_link"/>
-        </joint>
         <link name="${prefix}_base_link">
             <visual>
